File: PCB/pihpsdr Controller.kicad_pcb (KiCad board)
At the start: 2 copper layers, 238 x 154 mm, 161 parts, among them IC1 MCP23017T-E_SO, IC2 MCP23017T-E_SO, IC3 M24C32-RDW6TP, IC4 74LV1T125GVH, IC5 74LV1T125GVH, IC6 WM8960CGEFL_V, IC7 DS3231MZ_V+, J1 615008144221, J2 1725672, J3 485-1992, J4 SJ-3566AN, J6 10129379-905001BLF, J8 PJ-102AH, J9 MJ-3523-SMT, Q1 FDD6685, Q2 2N7002K, SW0 B3F-1055, SW1 B3F-1055, SW10 B3F-1055, SW11 B3F-1055, SW12 B3F-1055, SW13 B3F-1055, SW14 B3F-1055, SW15 B3F-1055, SW16 B3F-1055, SW2 B3F-1055, SW3 B3F-1055, SW4 B3F-1055, SW5 B3F-1055, SW6 B3F-1055, SW7 B3F-1055, SW8 B3F-1055, SW9 B3F-1055, U1 LMZ22005TZ_NOPB, U2 103, Y1 TSX-3225_24.0000MF18X-C

Commit message: Reorganized KiCad project
Parts:
- C18, C22: footprint SamacSys:CAPPM7343X310N -> SamacSys_Parts:CAPPM7343X310N
- C29, C32: footprint SamacSys:CAPPM6032X280N -> SamacSys_Parts:CAPPM6032X280N
- D2: footprint SamacSys:DIOM7959X262N -> SamacSys_Parts:DIOM7959X262N
- D3: footprint SamacSys:SODFL2512X80N -> SamacSys_Parts:SODFL2512X80N
- ENC1, J2: footprint SamacSys:1725672-4-2.54 -> SamacSys_Parts:1725672-4-2.54
- ENC2, ENC3, ENC4, ENC5: footprint SamacSys:EC11EBB24C03 -> SamacSys_Parts:EC11EBB24C03
- F1: footprint SamacSys:65600001009 -> SamacSys_Parts:65600001009
- IC1, IC2: footprint SamacSys:SOIC127P1030X265-28N -> SamacSys_Parts:SOIC127P1030X265-28N
- IC3: footprint SamacSys:SOP65P640X120-8N -> SamacSys_Parts:SOP65P640X120-8N
- IC4, IC5: footprint SamacSys:SOT95P275X110-5N -> SamacSys_Parts:SOT95P275X110-5N
- IC7: footprint SamacSys:SOIC127P600X175-8N -> SamacSys_Parts:SOIC127P600X175-8N
- J1: footprint SamacSys:615008144221 -> SamacSys_Parts:615008144221
- J3: footprint SamacSys:15445840_PI -> SamacSys_Parts:15445840_PI
- J6: footprint SamacSys:HDRRA5W67P0X254_1X5_1270X254X241P -> SamacSys_Parts:HDRRA5W67P0X254_1X5_1270X254X241P
- L1, L2, L3: footprint SamacSys:2743021447 -> SamacSys_Parts:2743021447
- Q1: footprint SamacSys:FQD1N80TM -> SamacSys_Parts:FQD1N80TM
- Q2: footprint SamacSys:SOT95P240X120-3N -> SamacSys_Parts:SOT95P240X120-3N
- SW0, SW1, SW10, SW11, SW12, SW13, SW14, SW15, SW16, SW2, SW3, SW4, SW5, SW6, SW7, SW8, SW9: footprint SamacSys:B3F1000 -> SamacSys_Parts:B3F1000
- U1: footprint SamacSys:NDW0007A -> SamacSys_Parts:NDW0007A
- U2: footprint SamacSys:103 -> SamacSys_Parts:103
- Y1: footprint SamacSys:TSX3225160000MF18XAC0 -> SamacSys_Parts:TSX3225160000MF18XAC0

Commit message: Cleaned up repository. Created a BOM in iBOM Format.
Parts:
- removed C3: 1µ, Capacitor_SMD:C_0805_2012Metric_Pad1.15x1.40mm_HandSolder
- added H11: MountingHole, MountingHole:MountingHole_3.2mm_M3_DIN965_Pad, F.Cu at (236.0, 112.0)
- added H9: MountingHole, MountingHole:MountingHole_3.2mm_M3_DIN965_Pad, F.Cu at (30.6, 134.0)
- added IC8: Pico, MCU_RaspberryPi_and_Boards:RPi_Pico_SMD_TH, B.Cu at (178.8, 75.4)
- added J5: SJ-3523-SMT-TR, CUI Devices:CUI_SJ-3523-SMT-TR, B.Cu at (28.5, 163.3)
- added J7: Conn_01x02, Connector_PinHeader_2.54mm:PinHeader_1x02_P2.54mm_Horizontal, B.Cu at (143.3, 117.4)
- added R66: 10k, Resistor_SMD:R_0805_2012Metric_Pad1.15x1.40mm_HandSolder, B.Cu at (42.4, 164.7)
- added R67: 10k, Resistor_SMD:R_0805_2012Metric_Pad1.15x1.40mm_HandSolder, B.Cu at (42.4, 160.6)
- J1: value 615008144221 -> 615008143721; footprint SamacSys_Parts:615008144221 -> SamacSys_Parts:615008143721
- R45, R46, R47, R48, R49: value R_Small -> 10k
- U2: value 103 -> BAT-HLD-001; footprint SamacSys_Parts:103 -> SamacSys_Parts:BATHLD001
- moved R12 106.0 mm to (55.0, 138.3), turned to 270 degrees
- moved R13 101.9 mm to (57.5, 138.3), turned to 270 degrees
- moved U2 91.5 mm to (127.6, 125.7)
- moved R11 88.9 mm to (80.0, 138.3), turned to 270 degrees
- moved IC7 80.2 mm to (88.4, 117.2)
- moved H5 27.6 mm to (30.6, 33.0)
- moved R15 22.8 mm to (214.5, 110.5)
- moved R3 22.8 mm to (217.1, 110.4)
- moved C15 22.8 mm to (212.4, 110.5)
- moved IC1 22.7 mm to (219.1, 119.0)
- moved J6 20.1 mm to (201.5, 50.9)
- moved C13 19.7 mm to (71.5, 51.4), turned to 270 degrees
- moved C4 15.5 mm to (56.4, 48.1), turned to 270 degrees
- moved Y1 15.1 mm to (67.4, 51.4), turned to 270 degrees
- moved C2 14.7 mm to (47.5, 52.0)
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Connections:
- C10 pad 1: Net-(C10-Pad1) -> GND
- C10 pad 2: +3V3 -> PI_3V3
- C11 pad 2: +3V3 -> PI_3V3
- C13 pad 1: +3V3 -> PI_3V3
- C35 pad 2: Net-(C35-Pad2) -> GND
- C5 pad 1: +3V3 -> PI_3V3
- C6 pad 2: +3V3 -> PI_3V3
- C9 pad 1: Net-(C10-Pad1) -> GND
- ENC2 pad A1: GPIO25 -> ENC2_A1
- ENC2 pad A2: GPIO23 -> ENC2_A2
- ENC2 pad B1: GPIO27 -> ENC2_B1
- ENC2 pad B2: GPIO26 -> ENC2_B2
- ENC3 pad A1: GPIO13 -> ENC3_A1
- ENC3 pad A2: GPIO14 -> ENC3_A2
- ENC3 pad B1: GPIO10 -> ENC3_B1
- ENC3 pad B2: GPIO11 -> ENC3_B2
- ENC4 pad A1: GPIO03 -> ENC4_A1
- ENC4 pad A2: GPIO06 -> ENC4_A2
- ENC4 pad B1: GPIO05 -> ENC4_B1
- ENC4 pad B2: GPIO12 -> ENC4_B2
- ENC5 pad A1: GPIO04 -> ENC5_A1
- ENC5 pad A2: GPIO02 -> ENC5_A2
- ENC5 pad B1: GPIO07 -> ENC5_B1
- ENC5 pad B2: GPIO00 -> ENC5_B2
- IC1 pad 12: SCL -> SCL1
- IC1 pad 13: SDA -> SDA1
- IC1 pad 20: IC2_INT -> IC1_INT
- IC2 pad 12: SCL -> SCL1
- IC2 pad 13: SDA -> SDA1
- IC2 pad 15: Net-(C35-Pad2) -> Net-(IC2-Pad15)
- IC2 pad 24: SW10 -> EXT_PTT
- IC2 pad 25: ENC4_BTN -> ENC2_BTN
- IC2 pad 27: ENC2_BTN -> ENC4_BTN
- IC2 pad 28: EXT_PTT -> SW10
- IC3 pad 8: +3V3 -> PI_3V3
- IC6 pad 10: +3V3 -> PI_3V3
- IC6 pad 21: +3V3 -> PI_3V3
- IC6 pad 26: +3V3 -> PI_3V3
- IC6 pad 28: Net-(C10-Pad1) -> GND
- IC6 pad 3: Net-(C2-Pad2) -> (no net)
- IC6 pad 32: +3V3 -> PI_3V3
- IC6 pad 4: Net-(C3-Pad2) -> Net-(C2-Pad2)
- IC6 pad 8: +3V3 -> PI_3V3
- IC7 pad 2: +3V3 -> PI_3V3
- J2 pad 3: SPK_R- -> SPK_R+
- J2 pad 4: SPK_R+ -> SPK_R-
- J3 pad 1: +3V3 -> PI_3V3
- J3 pad 10: IC2_INT -> PICO_TX
- J3 pad 11: GPIO00 -> (no net)
- J3 pad 13: GPIO02 -> (no net)
- J3 pad 15: GPIO03 -> (no net)
- J3 pad 16: GPIO04 -> (no net)
- J3 pad 17: +3V3 -> PI_3V3
- J3 pad 18: GPIO05 -> (no net)
- J3 pad 19: GPIO12 -> CW_SIDETONE
- J3 pad 21: GPIO13 -> CW_L
- J3 pad 22: GPIO06 -> (no net)
- J3 pad 23: GPIO14 -> CW_R
- J3 pad 24: GPIO10 -> (no net)
- J3 pad 26: GPIO11 -> (no net)
- J3 pad 29: ENC1- -> (no net)
- J3 pad 31: ENC1+ -> (no net)
- J3 pad 32: GPIO26 -> (no net)
- J3 pad 33: GPIO23 -> (no net)
- J3 pad 36: GPIO27 -> (no net)
- J3 pad 37: GPIO25 -> (no net)
- J3 pad 7: GPIO07 -> (no net)
- J3 pad 8: (no net) -> PICO_RX
- JP1 pad 2: +3V3 -> PI_3V3
- R1 pad 1: +3V3 -> PI_3V3
- R10 pad 1: +3V3 -> PI_3V3
- R17 pad 2: Net-(C35-Pad2) -> Net-(IC2-Pad15)
- R2 pad 1: +3V3 -> PI_3V3
- R27 pad 2: GPIO25 -> ENC2_A1
- R28 pad 2: GPIO27 -> ENC2_B1
- R29 pad 2: GPIO23 -> ENC2_A2
- R3 pad 2: IC2_INT -> IC1_INT
- R31 pad 2: GPIO26 -> ENC2_B2
- R32 pad 2: GPIO13 -> ENC3_A1
- R33 pad 2: GPIO10 -> ENC3_B1
- R34 pad 2: GPIO14 -> ENC3_A2
- R35 pad 2: GPIO11 -> ENC3_B2
- R36 pad 2: GPIO03 -> ENC4_A1
- R37 pad 2: GPIO05 -> ENC4_B1
- R38 pad 2: GPIO06 -> ENC4_A2
- R39 pad 2: GPIO12 -> ENC4_B2
- R40 pad 2: GPIO04 -> ENC5_A1
- R41 pad 2: GPIO07 -> ENC5_B1
- R42 pad 2: GPIO02 -> ENC5_A2
- R43 pad 2: GPIO00 -> ENC5_B2
- R63 pad 1: +3V3 -> PI_3V3
- R64 pad 1: +3V3 -> PI_3V3
- U2 pad 1: GND -> Net-(IC7-Pad6)
- Y1 pad 1: +3V3 -> PI_3V3
Routing:
- net +5V: track 164.0 -> 517.0 mm
- net PI_3V3: track 0.00 -> 302.0 mm, vias 0 -> 4
- net +3V3: track 511.5 -> 811.1 mm, vias 2 -> 4
- net SCL1: track 0.00 -> 228.0 mm, vias 0 -> 1
- net SDA1: track 0.00 -> 226.3 mm, vias 0 -> 1
- net SDA: track 63.1 -> 284.3 mm, vias 1 -> 4
- net SCL: track 66.3 -> 286.4 mm, vias 1 -> 4
- net ENC2_A1: track 0.00 -> 203.1 mm
- net ENC2_B1: track 0.00 -> 198.1 mm
- net ENC2_A2: track 0.00 -> 197.4 mm
- net ENC2_B2: track 0.00 -> 189.2 mm
- net ENC4_BTN: track 0.00 -> 172.6 mm, vias 0 -> 1
- net ENC3_A1: track 0.00 -> 169.0 mm
- net ENC3_A2: track 0.00 -> 166.3 mm
- net ENC3_B2: track 0.00 -> 159.1 mm
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Other:
- board size 238 x 154 mm -> 243 x 154 mm
- board text added: "+"
- board text added: "+5V"
- board text added: "-"
- board text added: "A"
- board text added: "B"
- board text added: "CW Sidetone Buzzer"
- board text added: "L+"
- board text added: "L-"
- board text added: "LC-Display"
- board text added: "R+"
- board text added: "R-"
- board text added: "Speaker"
- board text added: "VFO Encoder"
